File: 65HE_PCB.kicad_pcb (KiCad board)
At the start: 2 copper layers, 303.8 x 94.2 mm, 204 parts, among them J001 JST_SH, U1 SW_MX_HE, U10 SW_MX_HE, U11 SW_MX_HE, U12 SW_MX_HE, U13 SW_MX_HE, U14 SW_MX_HE, U15 SW_MX_HE, U16 SW_MX_HE, U17 SW_MX_HE, U18 SW_MX_HE, U19 SW_MX_HE, U2 SW_MX_HE, U20 SW_MX_HE, U201 XC6206PxxxMR, U202 TLV75733PDBV, U21 SW_MX_HE, U22 SW_MX_HE, U23 SW_MX_HE, U24 SW_MX_HE, U25 SW_MX_HE, U26 SW_MX_HE, U27 SW_MX_HE, U28 SW_MX_HE, U29 SW_MX_HE, U3 SW_MX_HE, U30 SW_MX_HE, U301 AT32F405CCT7, U31 SW_MX_HE, U32 SW_MX_HE, U33 SW_MX_HE, U34 SW_MX_HE, U35 SW_MX_HE, U36 SW_MX_HE, U37 SW_MX_HE, U38 SW_MX_HE, U39 SW_MX_HE, U4 SW_MX_HE, U40 SW_MX_HE, U41 SW_MX_HE, U42 SW_MX_HE, U43 SW_MX_HE, U44 SW_MX_HE, U45 SW_MX_HE, U46 SW_MX_HE, U47 SW_MX_HE, U48 SW_MX_HE, U49 SW_MX_HE, U5 SW_MX_HE, U50 SW_MX_HE, U51 SW_MX_HE, U52 SW_MX_HE, U53 SW_MX_HE, U54 SW_MX_HE, U55 SW_MX_HE, U56 SW_MX_HE, U57 SW_MX_HE, U58 SW_MX_HE, U59 SW_MX_HE, U6 SW_MX_HE, U60 SW_MX_HE, U61 SW_MX_HE, U62 SW_MX_HE, U63 SW_MX_HE, U64 SW_MX_HE, U65 SW_MX_HE, U66 SW_MX_HE, U67 SW_MX_HE, U68 SW_MX_HE, U69 SW_MX_HE, U7 SW_MX_HE, U70 SW_MX_HE, U71 SW_MX_HE, U72 SW_MX_HE, U73 SW_MX_HE, U74 SW_MX_HE, U75 SW_MX_HE, U8 SW_MX_HE, U9 SW_MX_HE, Y1 X322512MSB4SI

Commit message: full PCB and BOM
the pcb is done (i hope) and i made the production files and filled out the bom with parts from lcsc
Parts:
- renumbered C3 to C1, C12 to C10, C13 to C11, C14 to C12, C15 to C13, C1 to C14, C16 to C15, C2 to C16, C4 to C2, C5 to C3, C6 to C4, C7 to C5, C8 to C6, C71 to C63, C63 to C64, C72 to C65, C64 to C66, C73 to C67, C65 to C68, C74 to C69, C9 to C7, C66 to C70, C75 to C71, C67 to C72, C68 to C73, C69 to C74, C70 to C75, C10 to C8, C11 to C9, U3 to U1, U12 to U10, U13 to U11, U14 to U12, U15 to U13, U1 to U14, U16 to U15, U2 to U16, U4 to U2, U5 to U3, U6 to U4, U7 to U5, U8 to U6, U71 to U63, U63 to U64, U72 to U65, U64 to U66, U73 to U67, U65 to U68, U74 to U69, U9 to U7, U66 to U70, U75 to U71, U67 to U72, U68 to U73, U69 to U74, U70 to U75, U10 to U8, U11 to U9
Connections:
- AM501 pad 12: HE3 -> HE1
- AM501 pad 13: HE71 -> HE63
- AM501 pad 15: HE4 -> HE2
- AM502 pad 1: HE72 -> HE65
- AM502 pad 12: HE5 -> HE3
- AM502 pad 14: HE64 -> HE66
- AM502 pad 2: HE63 -> HE64
- AM503 pad 12: HE6 -> HE4
- AM503 pad 15: HE7 -> HE5
- AM503 pad 2: HE73 -> HE67
- AM504 pad 12: HE8 -> HE6
- AM505 pad 1: HE74 -> HE69
- AM505 pad 12: HE9 -> HE7
- AM505 pad 15: HE10 -> HE8
- AM505 pad 5: HE65 -> HE68
- AM506 pad 12: HE11 -> HE9
- AM506 pad 13: HE12 -> HE10
- AM507 pad 12: HE13 -> HE11
- AM507 pad 14: HE66 -> HE70
- AM508 pad 1: HE75 -> HE71
- AM508 pad 12: HE14 -> HE12
- AM508 pad 13: HE67 -> HE72
- AM509 pad 12: HE15 -> HE13
- AM509 pad 13: HE1 -> HE14
- AM509 pad 14: HE16 -> HE15
- AM509 pad 15: HE2 -> HE16
- AM509 pad 2: HE68 -> HE73
- AM510 pad 13: HE70 -> HE75
- AM510 pad 2: HE69 -> HE74
- U1 pad 2: HE3 -> HE1
- U10 pad 2: HE12 -> HE10
- U11 pad 2: HE13 -> HE11
- U12 pad 2: HE14 -> HE12
- U13 pad 2: HE15 -> HE13
- U14 pad 2: HE1 -> HE14
- U15 pad 2: HE16 -> HE15
- U16 pad 2: HE2 -> HE16
- U2 pad 2: HE4 -> HE2
- U3 pad 2: HE5 -> HE3
- U4 pad 2: HE6 -> HE4
- U5 pad 2: HE7 -> HE5
- U6 pad 2: HE8 -> HE6
- U63 pad 2: HE71 -> HE63
- U64 pad 2: HE63 -> HE64
- U65 pad 2: HE72 -> HE65
- U66 pad 2: HE64 -> HE66
- U67 pad 2: HE73 -> HE67
- U68 pad 2: HE65 -> HE68
- U69 pad 2: HE74 -> HE69
- U7 pad 2: HE9 -> HE7
- U70 pad 2: HE66 -> HE70
- U71 pad 2: HE75 -> HE71
- U72 pad 2: HE67 -> HE72
- U73 pad 2: HE68 -> HE73
- U74 pad 2: HE69 -> HE74
- U75 pad 2: HE70 -> HE75
- U8 pad 2: HE10 -> HE8
- U9 pad 2: HE11 -> HE9
Routing:
- net +3.3VA: track 1868.0 -> 1907.1 mm, vias 86 -> 87
- net HE2: track 30.7 -> 9.99 mm
- net HE12: track 20.8 -> 5.98 mm
- net HE10: track 9.99 -> 20.8 mm
- net HE16: track 21.7 -> 30.7 mm
- net HE6: track 14.8 -> 5.98 mm
- net HE3: track 14.8 -> 5.98 mm
- net HE9: track 14.8 -> 5.98 mm
- net HE72: track 68.9 -> 77.4 mm
- net HE73: track 75.2 -> 67.3 mm
- net HE63: track 70.7 -> 78.4 mm
- net HE15: track 14.8 -> 21.7 mm
- net HE14: track 5.98 -> 12.6 mm
- net HE11: track 5.98 -> 12.4 mm
- net HE71: track 78.4 -> 72.3 mm
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Other:
- outline, holes or cut-outs redrawn

Commit message: 1 less multiplexer!
made the whole board again to use only 1 sensor for each 1/8 unit pair of switches on the bottom row. i also made some improvements in the whole design itself
Parts:
- removed AM510: SN74LV4051A, Package_SO:TSSOP-16_4.4x5mm_P0.65mm
- removed C510: 100nF, Capacitor_SMD:C_0805_2012Metric
- removed the C63 at (82.0, 141.1)
- removed the C65 at (105.8, 141.1)
- removed the C67 at (129.6, 141.1)
- removed the C71 at (289.5, 141.1)
- removed the U63 at (81.0, 138.1)
- removed the U65 at (104.8, 138.1)
- removed the U67 at (128.6, 138.1)
- removed the U71 at (290.5, 138.1)
- U33: footprint PCM_marbastlib-he:SW_MX_HE_90deg_1u -> PCM_marbastlib-he:SW_MX_HE_90deg_1.75u_STP_1.25
- U62: footprint PCM_marbastlib-he:SW_MX_HE_90deg_NoVia -> PCM_marbastlib-he:SW_MX_HE_90deg_1_8u
- U63: renamed from U64; footprint PCM_marbastlib-he:SW_MX_HE_90deg_NoVia -> PCM_marbastlib-he:SW_MX_HE_90deg_1_8u
- U64: renamed from U66; footprint PCM_marbastlib-he:SW_MX_HE_90deg_NoVia -> PCM_marbastlib-he:SW_MX_HE_90deg_1_8u
- U68: renamed from U72; footprint PCM_marbastlib-he:SW_MX_HE_90deg_1u -> PCM_marbastlib-he:SW_MX_HE_90deg_1_8u
- moved AM509 38.1 mm to (352.4, 71.4), turned to -90 degrees
- moved D101 33.6 mm to (115.1, 105.6), turned to 90 degrees
- moved C306 28.9 mm to (106.8, 111.1), turned to 180 degrees
- moved C509 26.6 mm to (348.5, 75.4), turned to 90 degrees
- moved R302 22.9 mm to (106.8, 127.0), turned to 180 degrees
- moved NRST1 21.1 mm to (106.8, 115.5)
- moved BOOT0 20.8 mm to (106.8, 122.6), turned to 0 degrees
- moved AM501 19.1 mm to (104.8, 71.4), turned to -90 degrees
- moved AM503 19.1 mm to (161.9, 71.4), turned to -90 degrees
- moved AM504 19.1 mm to (190.5, 71.4), turned to -90 degrees
- moved AM506 19.1 mm to (247.7, 71.4), turned to -90 degrees
- moved AM507 19.1 mm to (276.2, 71.4), turned to -90 degrees
- moved AM508 19.1 mm to (304.8, 71.4), turned to -90 degrees
- moved AM502 19.0 mm to (133.3, 71.4), turned to -90 degrees
- moved AM505 19.0 mm to (219.1, 71.4), turned to -90 degrees
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- renumbered C64 to C63, C66 to C64, C68 to C65, C69 to C66, C70 to C67, C72 to C68, C73 to C69, C74 to C70, C75 to C71, U68 to U65, U69 to U66, U70 to U67, U73 to U69, U74 to U70, U75 to U71
Connections:
- AM501 pad 1: HE62 -> HE18
- AM501 pad 12: HE1 -> HE19
- AM501 pad 13: HE63 -> HE34
- AM501 pad 14: HE48 -> HE62
- AM501 pad 15: HE2 -> HE48
- AM501 pad 2: HE34 -> HE33
- AM501 pad 4: HE33 -> HE1
- AM501 pad 5: HE18 -> HE35
- AM502 pad 1: HE65 -> HE20
- AM502 pad 12: HE3 -> HE64
- AM502 pad 13: HE49 -> HE36
- AM502 pad 14: HE66 -> HE49
- AM502 pad 15: HE20 -> HE63
- AM502 pad 2: HE64 -> HE2
- AM502 pad 4: HE35 -> HE3
- AM502 pad 5: HE19 -> HE4
- AM503 pad 12: HE4 -> HE52
- AM503 pad 13: HE37 -> HE38
- AM503 pad 14: HE51 -> HE22
- AM503 pad 15: HE5 -> HE51
- AM503 pad 2: HE67 -> HE37
- AM503 pad 5: HE36 -> HE5
- AM504 pad 1: HE52 -> HE23
- AM504 pad 12: HE6 -> HE40
- AM504 pad 13: HE23 -> HE66
- AM504 pad 14: HE39 -> HE65
- AM504 pad 2: GND -> HE39
- AM504 pad 4: HE38 -> HE6
- AM504 pad 5: HE22 -> HE7
- AM505 pad 1: HE69 -> HE24
- AM505 pad 12: HE7 -> GND
- AM505 pad 13: HE54 -> HE55
- AM505 pad 14: GND -> HE41
- AM505 pad 15: HE8 -> HE25
- AM505 pad 2: HE40 -> HE54
- AM505 pad 4: HE24 -> HE8
- AM505 pad 5: HE68 -> HE9
- AM506 pad 1: HE55 -> HE26
- AM506 pad 12: HE9 -> HE43
- AM506 pad 13: HE10 -> HE57
- AM506 pad 14: HE42 -> HE67
- AM506 pad 15: HE26 -> HE56
- AM506 pad 2: GND -> HE42
- AM506 pad 4: HE41 -> HE10
- AM506 pad 5: HE25 -> HE27
- AM507 pad 1: HE56 -> HE11
- AM507 pad 12: HE11 -> HE68
- AM507 pad 13: HE43 -> HE58
- AM507 pad 14: HE70 -> HE44
- AM507 pad 15: HE57 -> HE28
- AM507 pad 2: GND -> HE12
- AM507 pad 4: HE27 -> HE45
- AM507 pad 5: GND -> HE29
- AM508 pad 1: HE71 -> HE13
- AM508 pad 12: HE12 -> HE46
- AM508 pad 13: HE72 -> HE30
- AM508 pad 14: HE29 -> HE69
- AM508 pad 15: HE45 -> HE59
- AM508 pad 2: HE58 -> HE14
- AM508 pad 4: HE44 -> HE15
- AM508 pad 5: HE28 -> HE16
- AM509 pad 1: HE46 -> HE31
- AM509 pad 12: HE13 -> HE47
- AM509 pad 13: HE14 -> HE71
- AM509 pad 14: HE15 -> HE61
- AM509 pad 15: HE16 -> HE70
- AM509 pad 2: HE73 -> HE60
- AM509 pad 4: HE30 -> HE17
- AM509 pad 5: HE59 -> HE32
- U301 pad 10: MUX_OUT_1 -> /ADC1_IN0
- U301 pad 11: MUX_OUT_2 -> MUX_OUT_1
- U301 pad 12: MUX_OUT_3 -> MUX_OUT_2
- U301 pad 13: MUX_OUT_4 -> MUX_OUT_3
- U301 pad 14: MUX_OUT_5 -> MUX_OUT_4
- U301 pad 15: MUX_OUT_6 -> MUX_OUT_5
- U301 pad 16: MUX_OUT_7 -> MUX_OUT_6
- U301 pad 17: MUX_OUT_8 -> MUX_OUT_7
- U301 pad 18: MUX_OUT_9 -> MUX_OUT_8
- U301 pad 19: MUX_OUT_10 -> MUX_OUT_9
- U301 pad 2: unconnected-(U301-PC13-Pad2) -> MUX_SEL_1
- U301 pad 3: unconnected-(U301-PC14-Pad3) -> MUX_SEL_2
- U301 pad 4: unconnected-(U301-PC15-Pad4) -> MUX_SEL_3
- U301 pad 41: MUX_SEL_1 -> unconnected-(U301-PB5-Pad41)
- U301 pad 42: MUX_SEL_2 -> unconnected-(U301-PB6-Pad42)
- U301 pad 43: MUX_SEL_3 -> unconnected-(U301-PB7-Pad43)
- U63 pad 2: HE64 -> HE63
- U64 pad 2: HE66 -> HE64
- U65 pad 2: HE68 -> HE65
- U66 pad 2: HE69 -> HE66
- U67 pad 2: HE70 -> HE67
- U68 pad 2: HE72 -> HE68
- U69 pad 2: HE73 -> HE69
- U70 pad 2: HE74 -> HE70
- U71 pad 2: HE75 -> HE71
Routing:
- net MUX_OUT_10: track 271.1 -> 0.00 mm, vias 2 -> 0
- net +3.3VA: track 1907.1 -> 1989.3 mm, vias 87 -> 81
- net HE72: track 77.4 -> 0.00 mm
- net HE75: track 75.0 -> 0.00 mm
- net HE73: track 67.3 -> 0.00 mm
- net HE74: track 67.1 -> 0.00 mm
- net MUX_OUT_9: track 233.3 -> 285.5 mm
- net MUX_OUT_5: track 118.1 -> 162.4 mm
- net MUX_SEL_3: track 335.4 -> 291.8 mm, vias 11 -> 10
- net MUX_OUT_3: track 57.8 -> 100.7 mm
- net MUX_OUT_4: track 86.2 -> 126.9 mm
- net MUX_OUT_2: track 28.2 -> 64.7 mm
- net MUX_OUT_8: track 201.7 -> 236.6 mm
- net HE2: track 9.99 -> 41.2 mm
- net MUX_SEL_2: track 324.9 -> 295.0 mm, vias 11 -> 10
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- removed copper zone on B.Cu, net +3.3V
Other:
- board text removed: "Boot"
- board text removed: "Connector"
- board text removed: "Reset"

Commit message: polished up the board and readme
added silckscreen to the board and filled out the readme with some basic information
Routing:
- net +3.3VA: track 1989.3 -> 1986.3 mm
- net HE20: track 14.1 -> 13.5 mm
- net GND: vias 1421 -> 1428
- net (no net): vias 7 -> 0
Other:
- board text added: "JST"
- board text added: "good luck future me"
- board text added: "hall effect analog keyboard pcb"
- board text added: "happy soldering!"
- board text added: "made by ZoharGalili"
- board text added: "the65HE"
- board text added: "this took so much time and effort to make"
