File: 65HE_PCB.kicad_pcb (KiCad board)
At the start: 2 copper layers, 303.8 x 94.2 mm, 194 parts, among them J001 JST_SH, U1 SW_MX_HE, U10 SW_MX_HE, U11 SW_MX_HE, U12 SW_MX_HE, U13 SW_MX_HE, U14 SW_MX_HE, U15 SW_MX_HE, U16 SW_MX_HE, U17 SW_MX_HE, U18 SW_MX_HE, U19 SW_MX_HE, U2 SW_MX_HE, U20 SW_MX_HE, U201 XC6206PxxxMR, U202 TLV75733PDBV, U21 SW_MX_HE, U22 SW_MX_HE, U23 SW_MX_HE, U24 SW_MX_HE, U25 SW_MX_HE, U26 SW_MX_HE, U27 SW_MX_HE, U28 SW_MX_HE, U29 SW_MX_HE, U3 SW_MX_HE, U30 SW_MX_HE, U301 AT32F405CCT7, U31 SW_MX_HE, U32 SW_MX_HE, U33 SW_MX_HE, U34 SW_MX_HE, U35 SW_MX_HE, U36 SW_MX_HE, U37 SW_MX_HE, U38 SW_MX_HE, U39 SW_MX_HE, U4 SW_MX_HE, U40 SW_MX_HE, U41 SW_MX_HE, U42 SW_MX_HE, U43 SW_MX_HE, U44 SW_MX_HE, U45 SW_MX_HE, U46 SW_MX_HE, U47 SW_MX_HE, U48 SW_MX_HE, U49 SW_MX_HE, U5 SW_MX_HE, U50 SW_MX_HE, U51 SW_MX_HE, U52 SW_MX_HE, U53 SW_MX_HE, U54 SW_MX_HE, U55 SW_MX_HE, U56 SW_MX_HE, U57 SW_MX_HE, U58 SW_MX_HE, U59 SW_MX_HE, U6 SW_MX_HE, U60 SW_MX_HE, U61 SW_MX_HE, U62 SW_MX_HE, U63 SW_MX_HE, U64 SW_MX_HE, U65 SW_MX_HE, U66 SW_MX_HE, U67 SW_MX_HE, U68 SW_MX_HE, U69 SW_MX_HE, U7 SW_MX_HE, U70 SW_MX_HE, U71 SW_MX_HE, U8 SW_MX_HE, U9 SW_MX_HE, Y1 X322512MSB4SI

Commit message: added test points
added test points to the pcb power lines and multiplexer outputs, hopefully the readme is fixed as well
Parts:
- added TP1: GND, TestPoint:TestPoint_Pad_2.0x2.0mm, B.Cu at (106.4, 92.9)
- added TP2: 3.3VA, TestPoint:TestPoint_Pad_D2.0mm, B.Cu at (103.6, 77.0)
- added TP3: 3.3V, TestPoint:TestPoint_Pad_D2.0mm, B.Cu at (93.3, 102.0)
- added TP501: AM1, TestPoint:TestPoint_Pad_D2.0mm, B.Cu at (108.7, 87.3)
- added TP502: AM2, TestPoint:TestPoint_Pad_D2.0mm, B.Cu at (138.9, 68.7)
- added TP503: AM3, TestPoint:TestPoint_Pad_D2.0mm, B.Cu at (167.5, 68.7)
- added TP504: AM4, TestPoint:TestPoint_Pad_D2.0mm, B.Cu at (196.1, 68.7)
- added TP505: AM5, TestPoint:TestPoint_Pad_D2.0mm, B.Cu at (224.6, 68.7)
- added TP506: AM6, TestPoint:TestPoint_Pad_D2.0mm, B.Cu at (244.5, 90.5)
- added TP507: AM7, TestPoint:TestPoint_Pad_D2.0mm, B.Cu at (270.7, 90.5)
- added TP508: AM8, TestPoint:TestPoint_Pad_D2.0mm, B.Cu at (298.8, 90.5)
- added TP509: AM9, TestPoint:TestPoint_Pad_D2.0mm, B.Cu at (358.0, 90.5)
Routing:
- net MUX_OUT_4: track 126.9 -> 129.7 mm
- net MUX_OUT_5: track 162.4 -> 165.2 mm
- net MUX_OUT_3: track 100.7 -> 103.5 mm
- net MUX_OUT_1: track 42.2 -> 44.9 mm
- net MUX_OUT_9: track 285.5 -> 288.3 mm
- net MUX_OUT_7: track 199.3 -> 202.1 mm
- net MUX_OUT_6: track 172.1 -> 174.9 mm
- net MUX_OUT_2: track 64.7 -> 67.3 mm
- net MUX_OUT_8: track 236.6 -> 238.9 mm
- net GND: track 40.9 -> 41.0 mm, vias 1428 -> 1419
Other:
- board text added: "Boot"
- board text added: "Reset"
